File: Schalterwerk/Gleisbelegung/gleis-a-2.brd (EAGLE design)
At the start: 100.3 x 80 mm, 55 parts, among them J1 PHNX_4P_508CONN_1017493, J2 PHNX_4P_508CONN_1017493, J3 PHNX_2P_508CONN_1017491, Q1 P-MOSFET, Q2 P-MOSFET, Q3 P-MOSFET, Q4 P-MOSFET, X2 IO-HAT, X4 RJ45-JACK, X5 PHNX_4P_350CONN_1984989_PXC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

Commit message: Renames signals on X4 again
Connections:
- net X41 renamed NX41
- net X42 renamed NX42
- net X43 renamed NX43
- net X44 renamed NX44
- net X45 renamed NX45
- net X46 renamed NX46
- net X47 renamed NX47
- net X48 renamed NX48
Changed lines of the file:
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@@
 <wire x1="67.31" y1="18.034" x2="67.31" y2="18.07600625" width="0.254" layer="16"/>
 </signal>
-<signal name="X41">
+<signal name="NX41">
 <contactref element="X4" pad="1"/>
 <contactref element="SJ9" pad="P$2"/>
@@
 <wire x1="12.954" y1="51.816" x2="12.954" y2="45.974" width="0.254" layer="1"/>
 </signal>
-<signal name="X42">
+<signal name="NX42">
 <contactref element="R9" pad="1"/>
 <contactref element="X4" pad="2"/>
@@
 <wire x1="13.208" y1="49.53" x2="18.1" y2="49.53" width="0.254" layer="16"/>
 </signal>
-<signal name="X43">
+<signal name="NX43">
 <contactref element="X4" pad="3"/>
 <contactref element="SJ9" pad="P$1"/>
@@
 <wire x1="10.922" y1="46.228" x2="16.637" y2="40.513" width="0.254" layer="16"/>
 </signal>
-<signal name="X45">
+<signal name="NX45">
 <contactref element="R11" pad="1"/>
 <contactref element="X4" pad="5"/>
@@
 <wire x1="7.254" y1="22.24" x2="5.08" y2="22.24" width="0.254" layer="16"/>
 </signal>
-<signal name="X47">
+<signal name="NX47">
 <contactref element="X4" pad="7"/>
 <contactref element="SJ11" pad="P$1"/>
@@
 <wire x1="21.844" y1="32.258" x2="21.844" y2="30.48" width="0.254" layer="16"/>
 </signal>
-<signal name="X48">
+<signal name="NX48">
 <contactref element="R12" pad="1"/>
 <contactref element="X4" pad="8"/>
@@
 <wire x1="25.4" y1="46.482" x2="25.4" y2="44.45" width="0.254" layer="16"/>
 </signal>
-<signal name="X46">
+<signal name="NX46">
 <contactref element="R10" pad="1"/>
 <contactref element="X4" pad="6"/>
@@
 <wire x1="25.4" y1="29.972" x2="25.4" y2="31.75" width="0.254" layer="16"/>
 </signal>
-<signal name="X44">
+<signal name="NX44">
 <contactref element="X4" pad="4"/>
 <contactref element="SJ10" pad="P$1"/>
