File: Schalterwerk/Weichen/weichen-a-5.brd (EAGLE design)
At the start: 63.5 x 80 mm, 50 parts, among them Q1 P-MOSFET, Q2 P-MOSFET, X1 PHNX_4P_508CONN_1017493, X2 IO-HAT, X3 PHNX_4P_350CONN_1984989_PXC, X4 PHNX_4P_350CONN_1984989_PXC, X5 RJ45-JACK

Commit message: Updates incorrect or inconsistent resistor values.
Parts:
- R1, R2: value 10k -> 5k
- R17, R18, R3, R4: value 5k -> 10k
Changed lines of the file:
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@@
 <attribute name="STANDARD" value="IPC-7351B" x="109.728" y="207.01" size="1.778" layer="28" rot="MR180" display="off"/>
 </element>
-<element name="R1" library="rcl" library_urn="urn:adsk.eagle:library:334" package="R0805" package3d_urn="urn:adsk.eagle:package:23553/2" value="10k" x="41.91" y="25.4" smashed="yes" rot="MR270">
+<element name="R1" library="rcl" library_urn="urn:adsk.eagle:library:334" package="R0805" package3d_urn="urn:adsk.eagle:package:23553/2" value="5k" x="41.91" y="25.4" smashed="yes" rot="MR270">
 <attribute name="NAME" x="42.418" y="23.114" size="1.27" layer="26" font="vector" ratio="10" rot="MR270"/>
 <attribute name="POPULARITY" value="86" x="209.55" y="-72.39" size="1.778" layer="28" rot="MR270" display="off"/>
@@
 <attribute name="SPICEPREFIX" value="R" x="110.49" y="194.31" size="1.778" layer="28" rot="MR180" display="off"/>
 </element>
-<element name="R2" library="rcl" library_urn="urn:adsk.eagle:library:334" package="R0805" package3d_urn="urn:adsk.eagle:package:23553/2" value="10k" x="41.91" y="35.56" smashed="yes" rot="MR270">
+<element name="R2" library="rcl" library_urn="urn:adsk.eagle:library:334" package="R0805" package3d_urn="urn:adsk.eagle:package:23553/2" value="5k" x="41.91" y="35.56" smashed="yes" rot="MR270">
 <attribute name="NAME" x="42.418" y="33.782" size="1.27" layer="26" font="vector" ratio="10" rot="MR270"/>
 <attribute name="POPULARITY" value="86" x="209.55" y="-67.31" size="1.778" layer="28" rot="MR270" display="off"/>
 <attribute name="SPICEPREFIX" value="R" x="209.55" y="-67.31" size="1.778" layer="28" rot="MR270" display="off"/>
 </element>
-<element name="R3" library="rcl" library_urn="urn:adsk.eagle:library:334" package="R0805" package3d_urn="urn:adsk.eagle:package:23553/2" value="5k" x="39.37" y="25.4" smashed="yes" rot="MR90">
+<element name="R3" library="rcl" library_urn="urn:adsk.eagle:library:334" package="R0805" package3d_urn="urn:adsk.eagle:package:23553/2" value="10k" x="39.37" y="25.4" smashed="yes" rot="MR90">
 <attribute name="NAME" x="39.878" y="23.114" size="1.27" layer="26" font="vector" ratio="10" rot="MR270"/>
 <attribute name="POPULARITY" value="86" x="-128.27" y="133.35" size="1.778" layer="28" rot="MR90" display="off"/>
 <attribute name="SPICEPREFIX" value="R" x="-128.27" y="133.35" size="1.778" layer="28" rot="MR90" display="off"/>
 </element>
-<element name="R4" library="rcl" library_urn="urn:adsk.eagle:library:334" package="R0805" package3d_urn="urn:adsk.eagle:package:23553/2" value="5k" x="39.37" y="35.56" smashed="yes" rot="MR90">
+<element name="R4" library="rcl" library_urn="urn:adsk.eagle:library:334" package="R0805" package3d_urn="urn:adsk.eagle:package:23553/2" value="10k" x="39.37" y="35.56" smashed="yes" rot="MR90">
 <attribute name="NAME" x="39.878" y="33.782" size="1.27" layer="26" font="vector" ratio="10" rot="MR270"/>
 <attribute name="POPULARITY" value="86" x="-128.27" y="148.59" size="1.778" layer="28" rot="MR90" display="off"/>
@@
 <attribute name="VALUE" x="59.563" y="31.75" size="1.27" layer="28" rot="MR90"/>
 </element>
-<element name="R17" library="rcl" library_urn="urn:adsk.eagle:library:334" package="R0805" package3d_urn="urn:adsk.eagle:package:23553/2" value="5k" x="57.912" y="31.242" smashed="yes" rot="MR0">
+<element name="R17" library="rcl" library_urn="urn:adsk.eagle:library:334" package="R0805" package3d_urn="urn:adsk.eagle:package:23553/2" value="10k" x="57.912" y="31.242" smashed="yes" rot="MR0">
 <attribute name="NAME" x="55.88" y="30.48" size="1.27" layer="26" font="vector" ratio="10" rot="MR0"/>
 <attribute name="POPULARITY" value="86" x="62.912" y="40.242" size="1.778" layer="28" rot="MR0" display="off"/>
@@
 <attribute name="NAME" x="38.862" y="4.318" size="1.27" layer="26" font="vector" ratio="10" rot="MR90"/>
 </element>
-<element name="R18" library="rcl" library_urn="urn:adsk.eagle:library:334" package="R0805" package3d_urn="urn:adsk.eagle:package:23553/2" value="5k" x="36.83" y="7.62" smashed="yes" rot="MR180">
+<element name="R18" library="rcl" library_urn="urn:adsk.eagle:library:334" package="R0805" package3d_urn="urn:adsk.eagle:package:23553/2" value="10k" x="36.83" y="7.62" smashed="yes" rot="MR180">
 <attribute name="NAME" x="34.925" y="10.16" size="1.27" layer="26" font="vector" ratio="10" rot="MR180"/>
 <attribute name="POPULARITY" value="86" x="17.83" y="5.62" size="1.778" layer="28" rot="MR180" display="off"/>
