File: Schalterwerk/screw-panel-front/screw-front-a-1.brd (EAGLE design)
At the start: 88.1 x 66 mm, 30 parts, among them J1 M4-SCREW-HOLE, J10 M4-SCREW-HOLE, J11 M4-SCREW-HOLE, J12 M4-SCREW-HOLE, J13 M4-SCREW-HOLE, J14 M4-SCREW-HOLE, J15 M4-SCREW-HOLE, J16 M4-SCREW-HOLE, J2 M4-SCREW-HOLE, J3 M4-SCREW-HOLE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

Commit message: Save files temporarily
Parts:
- added SJ1: (no value), eagleparts:SJ_RND2
- moved H2 56.7 mm to (4.83, 25.1)
- moved H1 47.0 mm to (4.83, 60.9)
- moved H3 29.0 mm to (44.9, 25.1)
- moved H4 19.1 mm to (44.9, 60.9)
Connections:
- net N$10: now also SJ1.P$1
- net N$9: now also SJ1.P$2
Routing:
- net N$10: track 0.00 -> 7.06 mm
- net N$9: track 0.00 -> 6.91 mm
Changed lines of the file:
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@@
 <setting verticaltext="up"/>
 </settings>
-<grid distance="1" unitdist="mm" unit="mm" style="lines" multiple="1" display="yes" altdistance="2" altunitdist="mil" altunit="mil"/>
+<grid distance="50" unitdist="mil" unit="mil" style="lines" multiple="1" display="yes" altdistance="2" altunitdist="mil" altunit="mil"/>
 <layers>
 <layer number="1" name="Top" color="4" fill="1" visible="yes" active="yes"/>
@@
 <wire x1="88" y1="66" x2="-0.12" y2="66" width="0" layer="20"/>
 <wire x1="-0.12" y1="66" x2="-0.12" y2="0" width="0" layer="20"/>
-<text x="39.464" y="58.184" size="1.27" layer="25" font="vector" ratio="10">(c) Balazs Racz
+<text x="5.816" y="33.464" size="1.27" layer="25" font="vector" ratio="10" rot="R90">(c) Balazs Racz
 20230617</text>
 <text x="11" y="63" size="1.778" layer="25">&gt;N01</text>
@@
 </autorouter>
 <elements>
-<element name="H1" library="holes" library_urn="urn:adsk.eagle:library:237" package="3,3" package3d_urn="urn:adsk.eagle:package:14278/1" value="MOUNT-HOLE3.3" x="47.833" y="41.93" smashed="yes" rot="MR0">
-<attribute name="POPULARITY" value="3" x="47.833" y="41.93" size="1.27" layer="28" font="vector" rot="MR0" display="off"/>
-</element>
-<element name="H2" library="holes" library_urn="urn:adsk.eagle:library:237" package="3,3" package3d_urn="urn:adsk.eagle:package:14278/1" value="MOUNT-HOLE3.3" x="60.833" y="34.08" smashed="yes" rot="MR0">
-<attribute name="POPULARITY" value="3" x="60.833" y="34.08" size="1.27" layer="28" font="vector" rot="MR0" display="off"/>
-</element>
-<element name="H3" library="holes" library_urn="urn:adsk.eagle:library:237" package="3,3" package3d_urn="urn:adsk.eagle:package:14278/1" value="MOUNT-HOLE3.3" x="65.92" y="5.08" smashed="yes" rot="MR0">
-<attribute name="POPULARITY" value="3" x="65.92" y="5.08" size="1.27" layer="28" font="vector" rot="MR0" display="off"/>
-</element>
-<element name="H4" library="holes" library_urn="urn:adsk.eagle:library:237" package="3,3" package3d_urn="urn:adsk.eagle:package:14278/1" value="MOUNT-HOLE3.3" x="63.92" y="58.93" smashed="yes" rot="MR0">
-<attribute name="POPULARITY" value="3" x="63.92" y="58.93" size="1.27" layer="28" font="vector" rot="MR0" display="off"/>
+<element name="H1" library="holes" library_urn="urn:adsk.eagle:library:237" package="3,3" package3d_urn="urn:adsk.eagle:package:14278/1" value="MOUNT-HOLE3.3" x="4.833" y="60.93" smashed="yes" rot="MR0">
+<attribute name="POPULARITY" value="3" x="4.833" y="60.93" size="1.27" layer="28" font="vector" rot="MR0" display="off"/>
+</element>
+<element name="H2" library="holes" library_urn="urn:adsk.eagle:library:237" package="3,3" package3d_urn="urn:adsk.eagle:package:14278/1" value="MOUNT-HOLE3.3" x="4.833" y="25.08" smashed="yes" rot="MR0">
+<attribute name="POPULARITY" value="3" x="4.833" y="25.08" size="1.27" layer="28" font="vector" rot="MR0" display="off"/>
+</element>
+<element name="H3" library="holes" library_urn="urn:adsk.eagle:library:237" package="3,3" package3d_urn="urn:adsk.eagle:package:14278/1" value="MOUNT-HOLE3.3" x="44.92" y="25.08" smashed="yes" rot="MR0">
+<attribute name="POPULARITY" value="3" x="44.92" y="25.08" size="1.27" layer="28" font="vector" rot="MR0" display="off"/>
+</element>
+<element name="H4" library="holes" library_urn="urn:adsk.eagle:library:237" package="3,3" package3d_urn="urn:adsk.eagle:package:14278/1" value="MOUNT-HOLE3.3" x="44.92" y="60.93" smashed="yes" rot="MR0">
+<attribute name="POPULARITY" value="3" x="44.92" y="60.93" size="1.27" layer="28" font="vector" rot="MR0" display="off"/>
 </element>
 <element name="J1" library="eagleparts" package="M4-SCREW-HOLE" value="M4-SCREW-HOLE" x="20" y="60" smashed="yes"/>
@@
 <attribute name="NAME" x="9.27" y="-62.92" size="1.27" layer="25" ratio="6"/>
 <attribute name="VALUE" x="9.27" y="-64.19" size="1.27" layer="27" ratio="6"/>
+</element>
+<element name="SJ1" library="eagleparts" package="SJ_RND2" value="" x="46.228" y="10.3632" smashed="yes" rot="R90">
+<attribute name="NAME" x="44.45" y="8.9662" size="1.27" layer="25" ratio="10" rot="R90"/>
 </element>
 </elements>
@@
 <contactref element="JP3" pad="2"/>
 <contactref element="JP3" pad="3"/>
-<wire x1="46.228" y1="15.748" x2="46.228" y2="13.208" width="0" layer="19" extent="1-1"/>
-<wire x1="46.228" y1="18.288" x2="46.228" y2="15.748" width="0" layer="19" extent="1-1"/>
+<wire x1="46.228" y1="18.288" x2="46.228" y2="15.748" width="0.8128" layer="1"/>
+<wire x1="46.228" y1="15.748" x2="46.228" y2="13.208" width="0.8128" layer="1"/>
+<contactref element="SJ1" pad="P$2"/>
+<wire x1="46.228" y1="13.208" x2="46.228" y2="11.42120625" width="0.8128" layer="1"/>
+<wire x1="46.228" y1="11.42120625" x2="46.22800625" y2="11.4212" width="0.8128" layer="1"/>
+<wire x1="46.228" y1="11.3792" x2="46.228" y2="11.42120625" width="0.508" layer="1"/>
 </signal>
 <signal name="N$10">
@@
 <contactref element="JP4" pad="2"/>
 <contactref element="JP4" pad="3"/>
-<wire x1="46.228" y1="5.588" x2="46.228" y2="3.048" width="0" layer="19" extent="1-1"/>
-<wire x1="46.228" y1="8.128" x2="46.228" y2="5.588" width="0" layer="19" extent="1-1"/>
+<wire x1="46.228" y1="3.048" x2="46.228" y2="5.588" width="0.8128" layer="1"/>
+<wire x1="46.228" y1="5.588" x2="46.228" y2="8.128" width="0.8128" layer="1"/>
+<contactref element="SJ1" pad="P$1"/>
+<wire x1="46.228" y1="8.128" x2="46.228" y2="10.1092" width="0.508" layer="1"/>
 </signal>
 <signal name="N$11">
