File: Schalterwerk/screw-panel-front/screw-front-a-1.sch (EAGLE design)
At the start: 26 parts, among them J1 M4-SCREW-HOLE, J10 M4-SCREW-HOLE, J11 M4-SCREW-HOLE, J12 M4-SCREW-HOLE, J13 M4-SCREW-HOLE, J14 M4-SCREW-HOLE, J15 M4-SCREW-HOLE, J16 M4-SCREW-HOLE, J2 M4-SCREW-HOLE, J3 M4-SCREW-HOLE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

Commit message: Save files temporarily
Parts:
- added SJ1: (no value), eagleparts:SJRND2
Connections:
- net N$10: now also SJ1.1
- net N$9: now also SJ1.2
Changed lines of the file:
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@@
 <part name="X3" library="eagleparts" deviceset="PHNX_4P_350" device="CONN_1984989_PXC"/>
 <part name="X4" library="eagleparts" deviceset="PHNX_4P_350" device="CONN_1984989_PXC"/>
+<part name="SJ1" library="eagleparts" deviceset="SJ" device="RND2"/>
 </parts>
 <sheets>
@@
 <attribute name="NAME" x="181.9646" y="124.6886" size="2.083" layer="95" ratio="6"/>
 </instance>
+<instance part="SJ1" gate="1" x="20.32" y="123.444" smashed="yes" rot="R90">
+<attribute name="NAME" x="17.78" y="120.904" size="1.778" layer="95" rot="R90"/>
+<attribute name="VALUE" x="24.13" y="120.904" size="1.778" layer="96" rot="R90"/>
+</instance>
 </instances>
 <busses>
@@
 <wire x1="25.4" y1="129.54" x2="33.02" y2="129.54" width="0.1524" layer="91"/>
 <junction x="25.4" y="132.08"/>
+<pinref part="SJ1" gate="1" pin="2"/>
+<wire x1="25.4" y1="132.08" x2="20.32" y2="132.08" width="0.1524" layer="91"/>
+<wire x1="20.32" y1="132.08" x2="20.32" y2="128.524" width="0.1524" layer="91"/>
 </segment>
 </net>
@@
 <wire x1="25.4" y1="111.76" x2="33.02" y2="111.76" width="0.1524" layer="91"/>
 <junction x="25.4" y="114.3"/>
-</segment>
-</net>
+<pinref part="SJ1" gate="1" pin="1"/>
+<wire x1="25.4" y1="114.3" x2="20.32" y2="114.3" width="0.1524" layer="91"/>
+<wire x1="20.32" y1="114.3" x2="20.32" y2="118.364" width="0.1524" layer="91"/>
+</segment>
+</net>
