File: Schalterwerk/screw-panel-front/screw-front-single-a-1.brd (EAGLE design)
At the start: 50 x 66 mm, 19 parts, among them J1 M4-SCREW-HOLE, J2 M4-SCREW-HOLE, J3 M4-SCREW-HOLE, J4 M4-SCREW-HOLE, J5 M4-SCREW-HOLE, J6 M4-SCREW-HOLE, J7 M4-SCREW-HOLE, J8 M4-SCREW-HOLE, X1 PHNX_4P_350CONN_1984989_PXC, X2 PHNX_4P_350CONN_1984989_PXC

Commit message: Adds alignment holes.
Parts:
- added H5, H6, H7: ALIGN-HOLE, eagleparts:ALIGNMENT-HOLE
Changed lines of the file:
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@@
 <layer number="113" name="ReferenceLS" color="7" fill="1" visible="no" active="no"/>
 <layer number="114" name="programming" color="7" fill="1" visible="no" active="yes"/>
+<layer number="115" name="laser-etch" color="47" fill="1" visible="no" active="yes"/>
 <layer number="116" name="Patch_BOT" color="9" fill="4" visible="no" active="yes"/>
+<layer number="117" name="laser-cut" color="63" fill="1" visible="yes" active="yes"/>
 <layer number="118" name="Rect_Pads" color="7" fill="1" visible="no" active="no"/>
 <layer number="121" name="_tsilk" color="7" fill="1" visible="no" active="yes"/>
@@
 <attribute name="NAME" x="49.45" y="8.9662" size="1.27" layer="25" ratio="10" rot="R90"/>
 </element>
+<element name="H5" library="eagleparts" package="ALIGNMENT-HOLE" value="ALIGN-HOLE" x="26" y="65" smashed="yes"/>
+<element name="H6" library="eagleparts" package="ALIGNMENT-HOLE" value="ALIGN-HOLE" x="1" y="21" smashed="yes"/>
+<element name="H7" library="eagleparts" package="ALIGNMENT-HOLE" value="ALIGN-HOLE" x="49" y="21" smashed="yes"/>
 </elements>
 <signals>
