File: Huenenberg/temp-stellwerk-a-3-laser-2.sch (EAGLE design)
At the start: 120 parts, among them Q1 BSS123, Q10 BSS84, Q11 BSS123, Q12 BSS84, Q13 BSS123, Q14 BSS84, Q15 BSS123, Q16 BSS84, Q17 BSS123, Q18 BSS84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

Commit message: Adds circles to laser around the tactile buttons.
Parts:
- H1, H2, H3: value MOUNT-HOLE3.2 -> MOUNT-HOLE4.0-LASER; device holes:MOUNT-HOLE3.2 -> eagleparts:MOUNT-HOLE4.0-LASER
- LOCK, TRK1, TRK2, TRK3, TRK4, TRK5, TRK6, W1, W1011, W2A, W2B, W34, W56, W7A, W7B, W89: device g-e2e-training:TACTSW-6X6S -> eagleparts:TACTSW-6X6S

Commit message: Adds laser holes on top of the LEDs.
Parts:
- DLOCK, DTRK1, DTRK2, DTRK3, DTRK4, DTRK5, DTRK6, DW1011N, DW1011N1, DW1011R, DW2BN, DW2BR, DW34N, DW34N1, DW34R, DW56N, DW56N1, DW56R, DW7BN, DW7BR, DW89N, DW89N1, DW89R: device led:LEDCHIP-LED0805 -> eagleparts:LEDCHIPLED_0805
- DW1N, DW1R, DW2AN, DW2AR, DW7AR: device led:LEDCHIP-LED0603 -> eagleparts:LEDCHIPLED_0603
