File: Huenenberg/temp-stellwerk-laser-4-left.sch (EAGLE design)
At the start: 120 parts, among them Q1 BSS123, Q10 BSS84, Q11 BSS123, Q12 BSS84, Q13 BSS123, Q14 BSS84, Q15 BSS123, Q16 BSS84, Q17 BSS123, Q18 BSS84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

Commit message: Adds final versions of lasered overlays.
Parts:
- LOCK: device trainlib:TACTSW-6X6S -> eagleparts:TACTSW-6X6S
Changed lines of the file:
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@@
 <part name="P+16" library="supply1" library_urn="urn:adsk.eagle:library:371" deviceset="+5V" device=""/>
 <part name="R43" library="rcl" library_urn="urn:adsk.eagle:library:334" deviceset="R-EU_" device="R0805" package3d_urn="urn:adsk.eagle:package:23553/2"/>
-<part name="LOCK" library="trainlib" deviceset="TACTSW-6X6" device="" technology="S" value="LOCK"/>
+<part name="LOCK" library="eagleparts" deviceset="TACTSW-6X6" device="" technology="S" value="LOCK"/>
 <part name="DLOCK" library="eagleparts" deviceset="LED" device="CHIPLED_0805" package3d_urn="urn:adsk.eagle:package:15821/2"/>
 <part name="Q25" library="eagleparts" deviceset="BSS123" device=""/>
