File: Block3/nucleo-block3-a-4.sch (EAGLE design)
At the start: 90 parts, among them IC2 TL331, J4 MODJACK6P6C-MJ3245-66-0CONN_M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, J5 MODJACK6P6C-MJ3245-66-0CONN_M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, Q1 NPN-23, Q3 BSS84, Q4 BSS123, U1 TC4428ACOA, U2 TC4428ACOA, U3 TC4428ACOA

Commit message: rearranges schematic sheets.
Parts:
- added R6: 47k, rcl:R-EU_R0805
Connections:
- net GND: now also R6.1
- net LN-TX-P: now also R6.2
Other:
- note added: "LN"
- note added: "Nucleo / LCC"
- note removed: "Digitalsystem"
Changed lines of the file:
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@@
 <attribute name="PAGE" value="LN port"/>
 </part>
+<part name="R6" library="rcl" library_urn="urn:adsk.eagle:library:334" deviceset="R-EU_" device="R0805" package3d_urn="urn:adsk.eagle:package:23553/2" value="47k"/>
 </parts>
 <sheets>
@@
 <wire x1="71.12" y1="180.34" x2="71.12" y2="55.88" width="0.1524" layer="97" style="longdash"/>
 <text x="66.04" y="182.88" size="1.778" layer="97">Isolierung</text>
-<text x="72.898" y="175.26" size="1.778" layer="97">Digitalsystem</text>
+<text x="72.898" y="175.26" size="1.778" layer="97">Nucleo / LCC</text>
 <wire x1="5.08" y1="55.88" x2="71.12" y2="55.88" width="0.1524" layer="97" style="longdash"/>
 <text x="175.26" y="-66.04" size="1.27" layer="91">Generates LN interrupt when
 TX=high and RX=low for 20 usec.</text>
 <wire x1="129.54" y1="-12.7" x2="129.54" y2="-142.24" width="0.1524" layer="97" style="longdash"/>
+<text x="124.46" y="-10.16" size="1.778" layer="97">Isolierung</text>
+<text x="121.92" y="-17.78" size="1.778" layer="97">LN</text>
+<text x="134.62" y="-17.78" size="1.778" layer="97">Nucleo / LCC</text>
 </plain>
 <instances>
@@
 <attribute name="VALUE" x="154.94" y="-50.8" size="1.778" layer="96" rot="MR0"/>
 </instance>
-<instance part="GND14" gate="1" x="157.48" y="-58.42" smashed="yes">
-<attribute name="VALUE" x="154.94" y="-60.96" size="1.778" layer="96"/>
+<instance part="GND14" gate="1" x="157.48" y="-60.96" smashed="yes">
+<attribute name="VALUE" x="154.94" y="-63.5" size="1.778" layer="96"/>
 </instance>
 <instance part="SUPPLY13" gate="G$1" x="119.38" y="-132.08" smashed="yes">
@@
 <attribute name="PAGE" x="161.29" y="-172.72" size="2.54" layer="94" font="vector"/>
 <attribute name="REVIEWER" x="176.53" y="-187.96" size="2.54" layer="94" font="vector"/>
+</instance>
+<instance part="R6" gate="G$1" x="165.1" y="-55.88" smashed="yes">
+<attribute name="NAME" x="163.83" y="-54.3814" size="1.778" layer="95"/>
+<attribute name="VALUE" x="163.83" y="-59.182" size="1.778" layer="96"/>
 </instance>
 </instances>
@@
 <pinref part="Q4" gate="N-CH" pin="S"/>
 <pinref part="GND14" gate="1" pin="GND"/>
+<wire x1="157.48" y1="-58.42" x2="157.48" y2="-55.88" width="0.1524" layer="91"/>
+<pinref part="R6" gate="G$1" pin="1"/>
 <wire x1="157.48" y1="-55.88" x2="157.48" y2="-53.34" width="0.1524" layer="91"/>
+<wire x1="160.02" y1="-55.88" x2="157.48" y2="-55.88" width="0.1524" layer="91"/>
+<junction x="157.48" y="-55.88"/>
 </segment>
 <segment>
@@
 <wire x1="149.86" y1="-40.64" x2="157.48" y2="-40.64" width="0.1524" layer="91"/>
 <pinref part="R47" gate="G$1" pin="2"/>
-<label x="165.1" y="-40.64" size="1.27" layer="95" xref="yes"/>
+<label x="177.8" y="-40.64" size="1.27" layer="95" xref="yes"/>
 <pinref part="Q4" gate="N-CH" pin="D"/>
-<wire x1="157.48" y1="-40.64" x2="165.1" y2="-40.64" width="0.1524" layer="91"/>
+<wire x1="157.48" y1="-40.64" x2="177.8" y2="-40.64" width="0.1524" layer="91"/>
 <wire x1="157.48" y1="-43.18" x2="157.48" y2="-40.64" width="0.1524" layer="91"/>
 <junction x="157.48" y="-40.64"/>
@@
 </segment>
 <segment>
-<wire x1="165.1" y1="-50.8" x2="162.56" y2="-50.8" width="0.1524" layer="91"/>
+<wire x1="177.8" y1="-50.8" x2="172.72" y2="-50.8" width="0.1524" layer="91"/>
 <pinref part="Q4" gate="N-CH" pin="G"/>
-<label x="165.1" y="-50.8" size="1.27" layer="95" xref="yes"/>
-</segment>
-</net>
+<label x="177.8" y="-50.8" size="1.27" layer="95" xref="yes"/>
+<pinref part="R6" gate="G$1" pin="2"/>
+<wire x1="172.72" y1="-50.8" x2="162.56" y2="-50.8" width="0.1524" layer="91"/>
+<wire x1="170.18" y1="-55.88" x2="172.72" y2="-55.88" width="0.1524" layer="91"/>
+<wire x1="172.72" y1="-55.88" x2="172.72" y2="-50.8" width="0.1524" layer="91"/>
+<junction x="172.72" y="-50.8"/>
+</segment>
+</net>

Commit message: Rearranges gates of the optocouplers.
Connections:
- net BLKA-RX-: now also OK2A.C, OK2B.A; no longer OK1A.C, OK1B.A
- net BLKC-RX-: now also OK1A.C, OK1B.A; no longer OK2A.C, OK2B.A
- net N$1: now also OK1A.A, OK1B.C; no longer OK2A.A, OK2B.C
- net N$2: now also OK1A.COL; no longer OK2A.COL
- net N$3: now also OK1B.COL; no longer OK2B.COL
- net N$31: now also OK2A.A, OK2B.C; no longer OK1A.A, OK1B.C
- net N$41: now also OK2A.COL; no longer OK1A.COL
- net N$42: now also OK2B.COL; no longer OK1B.COL
Other:
- moved on the sheet: OK1A, OK1B, OK2A, OK2B
Changed lines of the file:
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@@
 <attribute name="VALUE" x="195.5038" y="90.932" size="1.778" layer="96" rot="R90"/>
 </instance>
-<instance part="OK1" gate="A" x="73.66" y="165.1" smashed="yes">
+<instance part="OK2" gate="A" x="73.66" y="165.1" smashed="yes">
 <attribute name="NAME" x="66.675" y="170.815" size="1.778" layer="95"/>
 <attribute name="VALUE" x="66.675" y="157.48" size="1.778" layer="96"/>
 </instance>
-<instance part="OK1" gate="B" x="73.66" y="147.32" smashed="yes">
+<instance part="OK2" gate="B" x="73.66" y="147.32" smashed="yes">
 <attribute name="NAME" x="66.675" y="153.035" size="1.778" layer="95"/>
 <attribute name="VALUE" x="66.675" y="139.7" size="1.778" layer="96"/>
@@
 <attribute name="VALUE" x="107.315" y="94.615" size="1.778" layer="96"/>
 </instance>
-<instance part="OK2" gate="A" x="73.66" y="88.9" smashed="yes">
+<instance part="OK1" gate="A" x="73.66" y="88.9" smashed="yes">
 <attribute name="NAME" x="66.675" y="94.615" size="1.778" layer="95"/>
 <attribute name="VALUE" x="66.675" y="81.28" size="1.778" layer="96"/>
 </instance>
-<instance part="OK2" gate="B" x="73.66" y="71.12" smashed="yes">
+<instance part="OK1" gate="B" x="73.66" y="71.12" smashed="yes">
 <attribute name="NAME" x="66.675" y="76.835" size="1.778" layer="95"/>
 <attribute name="VALUE" x="66.675" y="63.5" size="1.778" layer="96"/>
@@
 <net name="GND" class="0">
 <segment>
-<pinref part="OK1" gate="A" pin="EMIT"/>
+<pinref part="OK2" gate="A" pin="EMIT"/>
 <wire x1="83.82" y1="162.56" x2="81.28" y2="162.56" width="0.1524" layer="91"/>
 <pinref part="GND1" gate="1" pin="GND"/>
 </segment>
 <segment>
-<pinref part="OK1" gate="B" pin="EMIT"/>
+<pinref part="OK2" gate="B" pin="EMIT"/>
 <pinref part="GND2" gate="1" pin="GND"/>
 <wire x1="83.82" y1="144.78" x2="81.28" y2="144.78" width="0.1524" layer="91"/>
@@
 </segment>
 <segment>
-<pinref part="OK2" gate="A" pin="EMIT"/>
+<pinref part="OK1" gate="A" pin="EMIT"/>
 <wire x1="83.82" y1="86.36" x2="81.28" y2="86.36" width="0.1524" layer="91"/>
 <pinref part="GND7" gate="1" pin="GND"/>
 </segment>
 <segment>
-<pinref part="OK2" gate="B" pin="EMIT"/>
+<pinref part="OK1" gate="B" pin="EMIT"/>
 <pinref part="GND8" gate="1" pin="GND"/>
 <wire x1="83.82" y1="68.58" x2="81.28" y2="68.58" width="0.1524" layer="91"/>
@@
 <net name="N$31" class="0">
 <segment>
-<pinref part="OK1" gate="A" pin="A"/>
+<pinref part="OK2" gate="A" pin="A"/>
 <pinref part="R9" gate="G$1" pin="1"/>
 <wire x1="63.5" y1="167.64" x2="58.42" y2="167.64" width="0.1524" layer="91"/>
-<pinref part="OK1" gate="B" pin="C"/>
+<pinref part="OK2" gate="B" pin="C"/>
 <wire x1="58.42" y1="167.64" x2="55.88" y2="167.64" width="0.1524" layer="91"/>
 <wire x1="63.5" y1="144.78" x2="58.42" y2="144.78" width="0.1524" layer="91"/>
@@
 <net name="BLKA-RX-" class="0">
 <segment>
-<pinref part="OK1" gate="B" pin="A"/>
+<pinref part="OK2" gate="B" pin="A"/>
 <wire x1="63.5" y1="149.86" x2="60.96" y2="149.86" width="0.1524" layer="91"/>
 <wire x1="60.96" y1="149.86" x2="60.96" y2="162.56" width="0.1524" layer="91"/>
-<pinref part="OK1" gate="A" pin="C"/>
+<pinref part="OK2" gate="A" pin="C"/>
 <wire x1="60.96" y1="162.56" x2="63.5" y2="162.56" width="0.1524" layer="91"/>
 <wire x1="60.96" y1="162.56" x2="40.64" y2="162.56" width="0.1524" layer="91"/>
@@
 <segment>
 <pinref part="R13" gate="G$1" pin="2"/>
-<pinref part="OK1" gate="A" pin="COL"/>
+<pinref part="OK2" gate="A" pin="COL"/>
 <wire x1="83.82" y1="167.64" x2="81.28" y2="167.64" width="0.1524" layer="91"/>
 </segment>
@@
 <segment>
 <pinref part="R14" gate="G$1" pin="2"/>
-<pinref part="OK1" gate="B" pin="COL"/>
+<pinref part="OK2" gate="B" pin="COL"/>
 <wire x1="83.82" y1="149.86" x2="81.28" y2="149.86" width="0.1524" layer="91"/>
 </segment>
@@
 <net name="N$1" class="0">
 <segment>
-<pinref part="OK2" gate="A" pin="A"/>
+<pinref part="OK1" gate="A" pin="A"/>
 <wire x1="63.5" y1="91.44" x2="58.42" y2="91.44" width="0.1524" layer="91"/>
-<pinref part="OK2" gate="B" pin="C"/>
+<pinref part="OK1" gate="B" pin="C"/>
 <wire x1="58.42" y1="91.44" x2="55.88" y2="91.44" width="0.1524" layer="91"/>
 <wire x1="63.5" y1="68.58" x2="58.42" y2="68.58" width="0.1524" layer="91"/>
@@
 <net name="BLKC-RX-" class="0">
 <segment>
-<pinref part="OK2" gate="B" pin="A"/>
+<pinref part="OK1" gate="B" pin="A"/>
 <wire x1="63.5" y1="73.66" x2="60.96" y2="73.66" width="0.1524" layer="91"/>
 <wire x1="60.96" y1="73.66" x2="60.96" y2="86.36" width="0.1524" layer="91"/>
-<pinref part="OK2" gate="A" pin="C"/>
+<pinref part="OK1" gate="A" pin="C"/>
 <wire x1="60.96" y1="86.36" x2="63.5" y2="86.36" width="0.1524" layer="91"/>
 <junction x="60.96" y="86.36"/>
@@
 <segment>
 <pinref part="R1" gate="G$1" pin="2"/>
-<pinref part="OK2" gate="A" pin="COL"/>
+<pinref part="OK1" gate="A" pin="COL"/>
 <wire x1="83.82" y1="91.44" x2="81.28" y2="91.44" width="0.1524" layer="91"/>
 </segment>
@@
 <segment>
 <pinref part="R2" gate="G$1" pin="2"/>
-<pinref part="OK2" gate="B" pin="COL"/>
+<pinref part="OK1" gate="B" pin="COL"/>
 <wire x1="83.82" y1="73.66" x2="81.28" y2="73.66" width="0.1524" layer="91"/>
 </segment>
