File: Block3/nucleo-block3-a-6.brd (EAGLE design)
At the start: 100.3 x 80 mm, 91 parts, among them IC1 TL331, J4 MODJACK6P6C-MJ3245-66-0CONN_M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, J5 MODJACK6P6C-MJ3245-66-0CONN_M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, Q1 NPN-23, Q2 BSS123, Q3 BSS84, U1 TC4428ACOA, U2 TC4428ACOA, U3 TC4428ACOA

Commit message: Routing the board.
Parts:
- R18: value 1200 -> 1k2
- U1, U2, U3: value TC4428ACOA -> TC4428
- moved SJ1 5.39 mm to (54.1, 31.5)
- moved R12 3.81 mm to (85.1, 21.6)
- moved R7 3.81 mm to (85.1, 17.8)
- moved R10 2.54 mm to (73.7, 39.4)
- moved R14 2.54 mm to (66.0, 39.4)
- moved R15 2.54 mm to (63.5, 39.4)
- moved R9 2.54 mm to (76.2, 39.4)
- moved R39 1.27 mm to (36.8, 55.9), turned to 0 degrees
- moved C7 0.81 mm to (19.7, 21.1)
- moved D3 0.51 mm to (16.5, 21.1)
- moved Q2 0.36 mm to (37.8, 65.8)
- moved R31 0.36 mm to (42.9, 65.8)
- moved D1 0.25 mm to (6.60, 33.7)
- turned LED7 to 180 degrees
- turned LED8 to 180 degrees
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Connections:
- net N$20 renamed LN-RX-ALT
- removed net 3V3: G1.3V3
- removed net GND3: G1.GND3
- removed net GND6: G1.GND6
- removed net GND7: G1.GND7
- new net VDD: G1.VDD
- net GND: now also G1.GND3, G1.GND6, G1.GND7
- net VCC: now also G1.3V3; no longer G1.VDD
Routing:
- net GND: track 0.00 -> 228.7 mm
- net +5V: track 0.00 -> 216.5 mm, vias 0 -> 3
- net BTNADC: track 0.00 -> 142.9 mm, vias 0 -> 9
- net AGND: track 0.00 -> 126.3 mm, vias 0 -> 6
- net VCC: track 0.00 -> 120.1 mm, vias 0 -> 7
- net LNPLUS: track 0.45 -> 118.6 mm, vias 0 -> 2
- net BLKA-TX+: track 0.00 -> 107.5 mm
- net BLKB-TX-: track 0.00 -> 98.1 mm
- net BLKA-TX-: track 0.00 -> 96.7 mm
- net N$14: track 0.00 -> 96.5 mm, vias 0 -> 2
- net BLKB-TX+: track 0.00 -> 86.6 mm
- net BLKB-RX: track 0.00 -> 84.9 mm, vias 0 -> 2
- net LN-TX: track 0.00 -> 77.6 mm, vias 0 -> 3
- net BLKC-RX-: track 0.00 -> 74.4 mm
- net LN-INT: track 0.00 -> 72.9 mm, vias 0 -> 4
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