File: Block3/nucleo-block3-a-7.brd (EAGLE design)
At the start: 100.3 x 80 mm, 91 parts, among them IC1 TL331, J4 MODJACK6P6C-MJ3245-66-0CONN_M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, J5 MODJACK6P6C-MJ3245-66-0CONN_M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, Q1 NPN-23, Q2 BSS123, Q3 BSS84, U1 TC4428, U2 TC4428, U3 TC4428

Commit message: Adds final routed board.
Parts:
- moved C1 1.00 mm to (72.1, 71.1)
- moved U2 1.00 mm to (75.9, 71.1)
- moved U3 1.00 mm to (67.0, 71.1)
Routing:
- net +5V: track 226.3 -> 221.1 mm
- net GND: track 511.9 -> 508.8 mm, vias 14 -> 113
- net BLKA-RX: track 59.4 -> 57.4 mm
- net BLKB-RX: track 87.1 -> 85.6 mm
- net BLKB-TX: track 71.7 -> 73.1 mm
- net BLKC-TX: track 68.7 -> 70.1 mm
- net BLKB-TX-: track 98.1 -> 97.1 mm
- net BLKC-TX-: track 65.9 -> 64.9 mm
- net BLKB-TX+: track 86.6 -> 85.6 mm
- net BLKC-TX+: track 64.6 -> 63.6 mm
- net LN-TX-B: track 55.4 -> 54.8 mm
- net LN-RX: track 71.9 -> 71.4 mm
Other:
- outline, holes or cut-outs redrawn
- board text added: "(c) Balazs Racz 20240505"
- board text added: "Anfangsf."
- board text added: "Block A"
- board text added: "Block B"
- board text added: "Block C"
- board text added: "Endfeld"
- board text added: "Erlaubnisf."
- board text added: "JP1: Power from LocoNet 2+3: Nucleo linear regulator 1+3: Switcher from LCC"
- board text added: "Nucleo-LN-Block3"
- board text added: "Rev. A7"
- board text removed: "(c) Balazs Racz 20240503"
- board text removed: ">REVISION"
- board text removed: "F1 RM"
- board text removed: "F2 RM"
- board text removed: "Fremo-LN-Block3"
- board text removed: "H RM"
- board text removed: "Masse"
- board text removed: "bl/w|"
- board text removed: "bl|"
- board text removed: "br/w|"
- board text removed: "br|"
- board text removed: "gn/w|"
- board text removed: "gn|"
- board text removed: "ora/w|"
- board text removed: "ora|"
