File: Block3/nucleo-block3-b-4.sch (EAGLE design)
At the start: 103 parts, among them IC1 TL331, IC2 ISO7221A, IC3 78L05F, J4 MODJACK6P6C-MJ3245-66-0CONN_M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, J5 MODJACK6P6C-MJ3245-66-0CONN_M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, Q1 NPN-23, Q2 BSS123, Q3 BSS84, Q4 BSS84, U1 TC4428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

Commit message: Final brd/sch that was ordered.
Parts:
- IC2: value ISO7221A -> ISO7721
Changed lines of the file:
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@@
 <part name="GND29" library="supply1" library_urn="urn:adsk.eagle:library:371" deviceset="GND" device=""/>
 <part name="P+1" library="supply1" library_urn="urn:adsk.eagle:library:371" deviceset="VCC" device=""/>
-<part name="IC2" library="texas" library_urn="urn:adsk.eagle:library:387" deviceset="ISO7221" device="" package3d_urn="urn:adsk.eagle:package:7566865/2" technology="A"/>
+<part name="IC2" library="texas" library_urn="urn:adsk.eagle:library:387" deviceset="ISO7221" device="" package3d_urn="urn:adsk.eagle:package:7566865/2" technology="A" value="ISO7721"/>
 <part name="IC3" library="linear" library_urn="urn:adsk.eagle:library:262" deviceset="78L*" device="F" package3d_urn="urn:adsk.eagle:package:16478/2" technology="05"/>
 <part name="SUPPLY7" library="supply2" library_urn="urn:adsk.eagle:library:372" deviceset="AGND" device=""/>
