File: Schalterwerk/Barrieren/barrieren-a-1.brd (EAGLE design)
At the start: 71.1 x 80 mm, 80 parts, among them Q1 BSS84, Q2 BSS84, Q3 BSS84, Q4 BSS84, Q5 BSS84, Q6 BSS84, X1 PHNX_4P_350CONN_1984989_PXC, X2 PHNX_4P_350CONN_1984989_PXC, X3 PHNX_4P_350CONN_1984989_PXC, X4 PHNX_4P_350CONN_1984989_PXC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

Commit message: Places connectors and adds labeling.
Parts:
- removed OK4, OK5, OK6, OK7, OK8: PC847, optocoupler:DIL16
- moved X2 94.1 mm to (5.08, 64.8), flipped to the bottom, turned to 90 degrees
- moved X1 44.5 mm to (5.08, 31.8), flipped to the bottom, turned to 90 degrees
- moved H4 14.0 mm to (19.1, 74.9)
- moved X3 6.35 mm to (5.08, 48.3)
Connections:
- net AGND: now also OK1.11, OK1.9; no longer OK3.13, OK3.15
- net GND: now also OK1.6, OK1.8, OK2.11, OK2.9, OK3.11, OK3.13, OK3.15, OK3.9; no longer OK1.11, OK3.2, OK3.4, OK4.11, OK5.11, OK6.11, OK7.11, OK8.11
- net N$10: now also OK1.5; no longer OK2.1
- net N$13: now also OK2.10; no longer OK4.12
- net N$15: now also OK3.1; no longer OK5.5
- net N$16: now also OK1.7; no longer OK2.3
- net N$19: now also OK2.16; no longer OK1.16
- net N$2: now also OK2.1; no longer OK1.1
- net N$20: now also OK3.16; no longer OK5.12
- net N$21: now also OK2.14; no longer OK1.14
- net N$23: now also OK3.3; no longer OK6.5
- net N$30: now also OK1.16; no longer OK3.16
- net N$31: now also OK2.12; no longer OK1.12
- net N$32: now also OK1.14; no longer OK3.14
- net N$33: now also OK1.1; no longer OK3.1
- net N$34: now also OK3.14; no longer OK6.12
- net N$35: now also OK1.3; no longer OK3.3
- net N$41: now also OK3.5; no longer OK7.5
- net N$43: now also OK3.12; no longer OK7.12
- net N$45: now also OK3.7; no longer OK8.5
- net N$47: now also OK3.10; no longer OK8.12
- net N$5: now also OK2.5; no longer OK1.5
- net N$6: now also OK1.12; no longer OK2.16
- net N$7: now also OK2.3; no longer OK1.3
- net N$8: now also OK2.7; no longer OK4.5
- net N$9: now also OK1.10; no longer OK2.14
- net NX3: now also OK2.8; no longer OK4.6
- net NX45: now also OK2.6; no longer OK1.6
- net NX6: now also OK3.2; no longer OK5.6
- net NX7: now also OK3.4; no longer OK6.6
- net NX8: now also OK3.6; no longer OK7.6
- net NX9: now also OK3.8; no longer OK8.6
Routing:
- net N$31: track 143.7 -> 0.00 mm, vias 5 -> 0
- net GND: track 105.9 -> 0.00 mm, vias 106 -> 0
- net N$28: track 97.7 -> 0.00 mm, vias 4 -> 0
- net N$25: track 74.1 -> 0.00 mm, vias 2 -> 0
- net AGND: track 47.5 -> 0.00 mm
- net NX45: track 34.0 -> 0.00 mm
- net +12V: track 29.0 -> 0.00 mm, vias 6 -> 0
- net NX41: track 25.0 -> 0.00 mm
- net N$4: track 22.4 -> 0.00 mm
- net N$5: track 17.9 -> 0.00 mm
- net NX43: track 17.5 -> 0.00 mm
- net N$11: track 16.0 -> 0.00 mm
- net +15V: track 13.4 -> 0.00 mm
- net N$7: track 9.95 -> 0.00 mm
- net N$2: track 4.66 -> 0.00 mm
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Other:
- board text added: "(c) Balazs Racz 20240601"
- board text added: "Barrierenadapter"
- board text removed: "(c) Balazs Racz 20230617"
- board text removed: "Farben nach 568B"
- board text removed: "IO board nach oben"
- board text removed: "L1"
- board text removed: "L2"
- board text removed: "L3"
- board text removed: "L4"
- board text removed: "Rückmelder"
- board text removed: "Weichenadapter"
- board text removed: "bl/w|"
- board text removed: "bl|"
- board text removed: "br/w|"
- board text removed: "br|"
- board text removed: "gn/w|"
- board text removed: "gn|"
- board text removed: "ora/w|"
- board text removed: "ora|"
