File: Schalterwerk/Barrieren/barrieren-a-2.brd (EAGLE design)
At the start: 71.1 x 80 mm, 75 parts, among them Q1 BSS84, Q2 BSS84, Q3 BSS84, Q4 BSS84, Q5 BSS84, Q6 BSS84, X1 PHNX_4P_350CONN_1984989_PXC, X2 PHNX_4P_350CONN_1984989_PXC, X3 PHNX_4P_350CONN_1984989_PXC, X4 PHNX_4P_350CONN_1984989_PXC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

Commit message: Continue on layout of barrieren board.
Parts:
- moved R27 228.6 mm to (28.0, 71.5)
- moved LED7 225.2 mm to (24.0, 75.0), turned to 270 degrees
- moved LED8 220.4 mm to (24.0, 71.5), turned to 90 degrees
- moved R19 217.1 mm to (29.3, 35.5)
- moved Q1 207.4 mm to (29.3, 38.5)
- moved R26 203.4 mm to (35.5, 69.5), turned to 180 degrees
- moved R25 197.9 mm to (17.0, 76.5), turned to 180 degrees
- moved OK3 178.9 mm to (42.0, 14.7), turned to 90 degrees
- moved LED9 170.6 mm to (24.0, 68.0), turned to 90 degrees
- moved LED10 165.7 mm to (24.0, 64.5), turned to 90 degrees
- moved OK2 156.4 mm to (43.3, 38.8), turned to 180 degrees
- moved R29 147.2 mm to (28.0, 68.0)
- moved R31 141.3 mm to (28.0, 64.5)
- moved LED11 52.2 mm to (24.0, 58.5), turned to 90 degrees
- moved R35 42.0 mm to (28.0, 55.0), turned to 0 degrees
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Routing:
- removed copper zone on layer 1, net GND
- removed copper zone on layer 16, net GND
Other:
- board text added: "RM B1:=-"
- board text added: "RM B1:=/"
- board text added: "RM B2:=-"
- board text added: "RM B2:=/"
- board text added: "RM B3:=-"
- board text added: "RM B3:=/"
- board text removed: "Ist+ schalt"
- board text removed: "Ist- schalt"
- board text removed: "Soll + RM"
- board text removed: "Soll - RM"

Commit message: Updates font and size of labels.
Parts:
- moved R27 11.1 mm to (17.0, 73.0), turned to 180 degrees
- moved R29 11.1 mm to (17.0, 69.5), turned to 180 degrees
- moved R31 11.1 mm to (17.0, 66.0), turned to 180 degrees
- moved R33 11.1 mm to (17.0, 60.0), turned to 180 degrees
- moved R35 11.1 mm to (17.0, 56.5), turned to 180 degrees
- moved R13 8.73 mm to (19.5, 44.0), turned to 180 degrees
- moved Q1 3.60 mm to (30.0, 42.0), turned to 90 degrees
- moved LED1 1.50 mm to (25.5, 42.0)
- moved LED10 0.50 mm to (24.5, 64.5), turned to 270 degrees
- moved LED11 0.50 mm to (24.5, 58.5), turned to 270 degrees
- moved LED12 0.50 mm to (24.5, 55.0), turned to 270 degrees
- moved LED7 0.50 mm to (24.5, 75.0)
- moved LED8 0.50 mm to (24.5, 71.5), turned to 270 degrees
- moved LED9 0.50 mm to (24.5, 68.0), turned to 270 degrees
Other:
- board text added: "917.01>B1:=/"
- board text added: "918.01<B1==-"
- board text added: "919.01>B1:=-"
- board text added: "925.01>B2:=-"
- board text added: "930.01>B3:=/"
- board text removed: "917.01 B1:=/"
- board text removed: "919.01 B1:=-"
- board text removed: "925.01 B2:=-"
- board text removed: "930.01 B3:=/"

Commit message: Finishes placing the components.
Parts:
- moved R6 316.1 mm to (52.1, 7.62), turned to 270 degrees
- moved R18 315.3 mm to (19.5, 23.5), turned to 180 degrees
- moved LED6 313.4 mm to (25.5, 22.0), turned to 270 degrees
- moved Q6 303.9 mm to (19.1, 16.5)
- moved R5 294.6 mm to (54.6, 7.62), turned to 270 degrees
- moved R17 294.3 mm to (19.5, 27.0), turned to 180 degrees
- moved R24 294.1 mm to (19.1, 11.4)
- moved R12 292.6 mm to (19.1, 7.62)
- moved LED5 292.3 mm to (25.5, 25.5), turned to 270 degrees
- moved Q5 282.1 mm to (24.1, 16.5)
- moved R16 275.9 mm to (19.5, 33.0), turned to 180 degrees
- moved LED4 274.1 mm to (25.5, 31.5), turned to 270 degrees
- moved R4 274.0 mm to (57.1, 7.62), turned to 270 degrees
- moved R23 271.8 mm to (24.1, 11.4)
- moved R11 270.7 mm to (24.1, 7.62)
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Connections:
- net B2-IS-CL-SCH: now also OK3.8; no longer OK3.2
- net B2-IS-OP-SCH: now also OK3.6; no longer OK3.4
- net B3-IS-CL-SCH: now also OK3.4; no longer OK3.6
- net B3-IS-OP-SCH: now also OK3.2; no longer OK3.8
- net N$15: now also OK3.7; no longer OK3.1
- net N$20: now also OK3.10; no longer OK3.16
- net N$23: now also OK3.5; no longer OK3.3
- net N$34: now also OK3.12; no longer OK3.14
- net N$41: now also OK3.3; no longer OK3.5
- net N$43: now also OK3.14; no longer OK3.12
- net N$45: now also OK3.1; no longer OK3.7
- net N$47: now also OK3.16; no longer OK3.10
Other:
- board text added: "918.01<B1==/"
- board text added: "920.01<B1==-"
- board text added: "921.01<B2==/"
- board text added: "922.01>B2:=/"
- board text added: "923.01<B2==-"
- board text added: "924.01<B3==/"
- board text added: "926.01<B3==-"
- board text added: "931.01>B3:=-"
- board text added: "Sch B1==-"
- board text added: "Sch B1==/"
- board text added: "Sch B2==-"
- board text added: "Sch B2==/"
- board text added: "Sch B3==-"
- board text added: "Sch B3==/"
- board text removed: "918.01<B1==-"
- board text removed: "922.01 B2:=/"
- board text removed: "931.01 B3:=-"
- board text removed: "Schaltdecoder"
