File: Schalterwerk/Barrieren/barrieren-a-2.sch (EAGLE design)
At the start: 71 parts, among them Q1 BSS84, Q2 BSS84, Q3 BSS84, Q4 BSS84, Q5 BSS84, Q6 BSS84, X1 PHNX_4P_350CONN_1984989_PXC, X2 PHNX_4P_350CONN_1984989_PXC, X3 PHNX_4P_350CONN_1984989_PXC, X4 PHNX_4P_350CONN_1984989_PXC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

Commit message: Finishes placing the components.
Connections:
- net B2-IS-CL-SCH: now also OK3D.C; no longer OK3A.C
- net B2-IS-OP-SCH: now also OK3C.C; no longer OK3B.C
- net B3-IS-CL-SCH: now also OK3B.C; no longer OK3C.C
- net B3-IS-OP-SCH: now also OK3A.C; no longer OK3D.C
- net N$15: now also OK3D.A; no longer OK3A.A
- net N$20: now also OK3D.COL; no longer OK3A.COL
- net N$23: now also OK3C.A; no longer OK3B.A
- net N$34: now also OK3C.COL; no longer OK3B.COL
- net N$41: now also OK3B.A; no longer OK3C.A
- net N$43: now also OK3B.COL; no longer OK3C.COL
- net N$45: now also OK3A.A; no longer OK3D.A
- net N$47: now also OK3A.COL; no longer OK3D.COL
Other:
- moved on the sheet: OK3A, OK3B, OK3C, OK3D
Changed lines of the file:
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@@
 <attribute name="VALUE" x="35.56" y="155.575" size="1.778" layer="96" rot="MR0"/>
 </instance>
-<instance part="OK3" gate="A" x="58.42" y="124.46" smashed="yes">
+<instance part="OK3" gate="D" x="58.42" y="124.46" smashed="yes">
 <attribute name="NAME" x="51.435" y="130.175" size="1.778" layer="95"/>
 <attribute name="VALUE" x="51.435" y="116.84" size="1.778" layer="96"/>
@@
 <attribute name="VALUE" x="35.56" y="132.715" size="1.778" layer="96" rot="MR0"/>
 </instance>
-<instance part="OK3" gate="B" x="58.42" y="101.6" smashed="yes">
+<instance part="OK3" gate="C" x="58.42" y="101.6" smashed="yes">
 <attribute name="NAME" x="51.435" y="107.315" size="1.778" layer="95"/>
 <attribute name="VALUE" x="51.435" y="93.98" size="1.778" layer="96"/>
@@
 <attribute name="VALUE" x="35.56" y="109.855" size="1.778" layer="96" rot="MR0"/>
 </instance>
-<instance part="OK3" gate="C" x="58.42" y="78.74" smashed="yes">
+<instance part="OK3" gate="B" x="58.42" y="78.74" smashed="yes">
 <attribute name="NAME" x="51.435" y="84.455" size="1.778" layer="95"/>
 <attribute name="VALUE" x="51.435" y="71.12" size="1.778" layer="96"/>
@@
 <attribute name="VALUE" x="35.56" y="86.995" size="1.778" layer="96" rot="MR0"/>
 </instance>
-<instance part="OK3" gate="D" x="58.42" y="55.88" smashed="yes">
+<instance part="OK3" gate="A" x="58.42" y="55.88" smashed="yes">
 <attribute name="NAME" x="51.435" y="61.595" size="1.778" layer="95"/>
 <attribute name="VALUE" x="51.435" y="48.26" size="1.778" layer="96"/>
@@
 </segment>
 <segment>
-<pinref part="OK3" gate="A" pin="EMIT"/>
+<pinref part="OK3" gate="D" pin="EMIT"/>
 <wire x1="66.04" y1="121.92" x2="68.58" y2="121.92" width="0.1524" layer="91"/>
 <pinref part="GND11" gate="1" pin="GND"/>
@@
 </segment>
 <segment>
-<pinref part="OK3" gate="B" pin="EMIT"/>
+<pinref part="OK3" gate="C" pin="EMIT"/>
 <wire x1="66.04" y1="99.06" x2="68.58" y2="99.06" width="0.1524" layer="91"/>
 <pinref part="GND12" gate="1" pin="GND"/>
@@
 </segment>
 <segment>
-<pinref part="OK3" gate="C" pin="EMIT"/>
+<pinref part="OK3" gate="B" pin="EMIT"/>
 <wire x1="66.04" y1="76.2" x2="68.58" y2="76.2" width="0.1524" layer="91"/>
 <pinref part="GND13" gate="1" pin="GND"/>
@@
 </segment>
 <segment>
-<pinref part="OK3" gate="D" pin="EMIT"/>
+<pinref part="OK3" gate="A" pin="EMIT"/>
 <wire x1="66.04" y1="53.34" x2="68.58" y2="53.34" width="0.1524" layer="91"/>
 <pinref part="GND14" gate="1" pin="GND"/>
@@
 <net name="B2-IS-CL-SCH" class="0">
 <segment>
-<pinref part="OK3" gate="A" pin="C"/>
+<pinref part="OK3" gate="D" pin="C"/>
 <pinref part="X1" gate="A" pin="2"/>
 <wire x1="48.26" y1="121.92" x2="15.24" y2="121.92" width="0.1524" layer="91"/>
@@
 <segment>
 <pinref part="R3" gate="G$1" pin="2"/>
-<pinref part="OK3" gate="A" pin="A"/>
+<pinref part="OK3" gate="D" pin="A"/>
 <wire x1="45.72" y1="127" x2="48.26" y2="127" width="0.1524" layer="91"/>
 </segment>
@@
 <net name="N$20" class="0">
 <segment>
-<pinref part="OK3" gate="A" pin="COL"/>
+<pinref part="OK3" gate="D" pin="COL"/>
 <wire x1="68.58" y1="127" x2="66.04" y2="127" width="0.1524" layer="91"/>
 <pinref part="LED3" gate="G$1" pin="C"/>
@@
 <net name="B2-IS-OP-SCH" class="0">
 <segment>
-<pinref part="OK3" gate="B" pin="C"/>
+<pinref part="OK3" gate="C" pin="C"/>
 <pinref part="X1" gate="A" pin="1"/>
 <wire x1="48.26" y1="99.06" x2="12.7" y2="99.06" width="0.1524" layer="91"/>
@@
 <segment>
 <pinref part="R4" gate="G$1" pin="2"/>
-<pinref part="OK3" gate="B" pin="A"/>
+<pinref part="OK3" gate="C" pin="A"/>
 <wire x1="45.72" y1="104.14" x2="48.26" y2="104.14" width="0.1524" layer="91"/>
 </segment>
@@
 <net name="N$34" class="0">
 <segment>
-<pinref part="OK3" gate="B" pin="COL"/>
+<pinref part="OK3" gate="C" pin="COL"/>
 <wire x1="68.58" y1="104.14" x2="66.04" y2="104.14" width="0.1524" layer="91"/>
 <pinref part="LED4" gate="G$1" pin="C"/>
@@
 <net name="B3-IS-CL-SCH" class="0">
 <segment>
-<pinref part="OK3" gate="C" pin="C"/>
+<pinref part="OK3" gate="B" pin="C"/>
 <pinref part="X2" gate="A" pin="4"/>
 <wire x1="48.26" y1="76.2" x2="12.7" y2="76.2" width="0.1524" layer="91"/>
@@
 <segment>
 <pinref part="R5" gate="G$1" pin="2"/>
-<pinref part="OK3" gate="C" pin="A"/>
+<pinref part="OK3" gate="B" pin="A"/>
 <wire x1="45.72" y1="81.28" x2="48.26" y2="81.28" width="0.1524" layer="91"/>
 </segment>
@@
 <net name="N$43" class="0">
 <segment>
-<pinref part="OK3" gate="C" pin="COL"/>
+<pinref part="OK3" gate="B" pin="COL"/>
 <wire x1="68.58" y1="81.28" x2="66.04" y2="81.28" width="0.1524" layer="91"/>
 <pinref part="LED5" gate="G$1" pin="C"/>
@@
 <net name="B3-IS-OP-SCH" class="0">
 <segment>
-<pinref part="OK3" gate="D" pin="C"/>
+<pinref part="OK3" gate="A" pin="C"/>
 <pinref part="X2" gate="A" pin="3"/>
 <wire x1="48.26" y1="53.34" x2="15.24" y2="53.34" width="0.1524" layer="91"/>
@@
 <segment>
 <pinref part="R6" gate="G$1" pin="2"/>
-<pinref part="OK3" gate="D" pin="A"/>
+<pinref part="OK3" gate="A" pin="A"/>
 <wire x1="45.72" y1="58.42" x2="48.26" y2="58.42" width="0.1524" layer="91"/>
 </segment>
@@
 <net name="N$47" class="0">
 <segment>
-<pinref part="OK3" gate="D" pin="COL"/>
+<pinref part="OK3" gate="A" pin="COL"/>
 <wire x1="68.58" y1="58.42" x2="66.04" y2="58.42" width="0.1524" layer="91"/>
 <pinref part="LED6" gate="G$1" pin="C"/>
